Commit message: improved urdf visual, added com for base link

File: visualize_ur/ur4_description/simple_geometry.urdf (robot description, URDF)
Before this commit: robot simple_geometry, 3 links, 2 joints
Links:
- link base_link: mass None -> 10
- link shoulder_link: geometry collision cylinder length=0.1 radius=0.15; visual cylinder length=0.1 radius=0.15
Joints:
- joint shoulder_pan_joint: origin xyz=0.0 0.0 0.089159 rpy=0.0 0.0 0.0 -> xyz=0.0 0.0 0.1 rpy=0.0 0.0 0.0
