Commit message: removed unuseful fixed joint from the UR4 robot
added some comments in the code

File: visualize_ur/ur4_description/ur4_robot.urdf (robot description, URDF)
Before this commit: robot ur5, 8 links, 7 joints
Links:
- removed link base
Joints:
- removed joint base_link-base_fixed_joint
