Commit message: added solo12 support

File: robot_urdf/solo12.urdf (robot description, URDF)
Before this commit: robot solo, 20 links, 19 joints
Links:
- removed link FL_foot
- removed link FL_hip_assembly
- removed link FL_lower_leg
- removed link FL_upper_leg
- removed link FR_foot
- removed link FR_hip_assembly
- removed link FR_lower_leg
- removed link FR_upper_leg
- removed link HL_foot
- removed link HL_hip_assembly
- removed link HL_lower_leg
- removed link HL_upper_leg
- removed link HR_foot
- removed link HR_hip_assembly
- removed link HR_lower_leg
- removed link HR_upper_leg
- removed link base_inertia
- added link lf_foot, mass 0.00693606; collision mesh filename=package://solo_description/meshes/stl/with_foot/solo_foot.s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; visual mesh filename=package://solo_description/meshes/stl/with_foot/solo_foot.s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
- added link lf_hip_assembly, mass 0.150
- added link lf_lower_leg, mass 0.03070001; collision mesh filename=package://solo_description/meshes/stl/with_foot/solo_lower_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; visual mesh filename=package://solo_description/meshes/stl/with_foot/solo_lower_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
- added link lf_upper_leg, mass 0.14853845; collision mesh filename=package://solo_description/meshes/stl/with_foot/solo_upper_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; visual mesh filename=package://solo_description/meshes/stl/with_foot/solo_upper_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
- added link lh_foot, mass 0.00693606; collision mesh filename=package://solo_description/meshes/stl/with_foot/solo_foot.s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; visual mesh filename=package://solo_description/meshes/stl/with_foot/solo_foot.s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
- added link lh_hip_assembly, mass 0.150
- added link lh_lower_leg, mass 0.03070001; collision mesh filename=package://solo_description/meshes/stl/with_foot/solo_lower_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; visual mesh filename=package://solo_description/meshes/stl/with_foot/solo_lower_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
- added link lh_upper_leg, mass 0.14853845; collision mesh filename=package://solo_description/meshes/stl/with_foot/solo_upper_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; visual mesh filename=package://solo_description/meshes/stl/with_foot/solo_upper_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
- added link rf_foot, mass 0.00693606; collision mesh filename=package://solo_description/meshes/stl/with_foot/solo_foot.s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; visual mesh filename=package://solo_description/meshes/stl/with_foot/solo_foot.s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
- added link rf_hip_assembly, mass 0.150
- added link rf_lower_leg, mass 0.03070001; collision mesh filename=package://solo_description/meshes/stl/with_foot/solo_lower_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; visual mesh filename=package://solo_description/meshes/stl/with_foot/solo_lower_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
- added link rf_upper_leg, mass 0.14853845; collision mesh filename=package://solo_description/meshes/stl/with_foot/solo_upper_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; visual mesh filename=package://solo_description/meshes/stl/with_foot/solo_upper_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
- added link rh_foot, mass 0.00693606; collision mesh filename=package://solo_description/meshes/stl/with_foot/solo_foot.s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; visual mesh filename=package://solo_description/meshes/stl/with_foot/solo_foot.s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
- added link rh_hip_assembly, mass 0.150
- added link rh_lower_leg, mass 0.03070001; collision mesh filename=package://solo_description/meshes/stl/with_foot/solo_lower_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; visual mesh filename=package://solo_description/meshes/stl/with_foot/solo_lower_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
- added link rh_upper_leg, mass 0.14853845; collision mesh filename=package://solo_description/meshes/stl/with_foot/solo_upper_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; visual mesh filename=package://solo_description/meshes/stl/with_foot/solo_upper_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
- link base_link: geometry 
- link trunk: mass None -> 1.63315091; geometry collision mesh filename=package://solo_description/meshes/stl/with_foot/solo_body.s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; visual mesh filename=package://solo_description/meshes/stl/with_foot/solo_body.s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
Joints:
- removed joint FL_ankle
- removed joint FL_haa_joint
- removed joint FL_hfe_joint
- removed joint FL_kfe_joint
- removed joint FR_ankle
- removed joint FR_haa_joint
- removed joint FR_hfe_joint
- removed joint FR_kfe_joint
- removed joint HL_ankle
- removed joint HL_haa_joint
- removed joint HL_hfe_joint
- removed joint HL_kfe_joint
- removed joint HR_ankle
- removed joint HR_haa_joint
- removed joint HR_hfe_joint
- removed joint HR_kfe_joint
- removed joint base_to_base_inertia
- added joint lf_ankle: type fixed, parent lf_lower_leg, child lf_foot, origin xyz=0 0 -0.16 rpy=0 0 0, limit lower=-10 upper=10 effort=1000 velocity=1000
- added joint lf_haa_joint: type revolute, parent trunk, child lf_hip_assembly, origin xyz=0.19 0.1046 0 rpy=0 0 0, axis 1 0 0, limit lower=-10 upper=10 effort=1000 velocity=1000
- added joint lf_hfe_joint: type revolute, parent lf_hip_assembly, child lf_upper_leg, origin xyz=0 0 0 rpy=0 0 0, axis 0 1 0, limit lower=-10 upper=10 effort=1000 velocity=1000
- added joint lf_kfe_joint: type revolute, parent lf_upper_leg, child lf_lower_leg, origin xyz=0 0.03745 -0.16 rpy=0 0 0, axis 0 1 0, limit lower=-10 upper=10 effort=1000 velocity=1000
- added joint lh_ankle: type fixed, parent lh_lower_leg, child lh_foot, origin xyz=0 0 -0.16 rpy=0 0 0, limit lower=-10 upper=10 effort=1000 velocity=1000
- added joint lh_haa_joint: type revolute, parent trunk, child lh_hip_assembly, origin xyz=-0.19 0.1046 0 rpy=0 0 0, axis 1 0 0, limit lower=-10 upper=10 effort=1000 velocity=1000
- added joint lh_hfe_joint: type revolute, parent lh_hip_assembly, child lh_upper_leg, origin xyz=0 0 0 rpy=0 0 0, axis 0 1 0, limit lower=-10 upper=10 effort=1000 velocity=1000
- added joint lh_kfe_joint: type revolute, parent lh_upper_leg, child lh_lower_leg, origin xyz=0 0.03745 -0.16 rpy=0 0 0, axis 0 1 0, limit lower=-10 upper=10 effort=1000 velocity=1000
- added joint rf_ankle: type fixed, parent rf_lower_leg, child rf_foot, origin xyz=0 0 -0.16 rpy=0 0 0, limit lower=-10 upper=10 effort=1000 velocity=1000
- added joint rf_haa_joint: type revolute, parent trunk, child rf_hip_assembly, origin xyz=0.19 -0.1046 0 rpy=0 0 0, axis 1 0 0, limit lower=-10 upper=10 effort=1000 velocity=1000
- added joint rf_hfe_joint: type revolute, parent rf_hip_assembly, child rf_upper_leg, origin xyz=0 0 0 rpy=0 0 0, axis 0 1 0, limit lower=-10 upper=10 effort=1000 velocity=1000
- added joint rf_kfe_joint: type revolute, parent rf_upper_leg, child rf_lower_leg, origin xyz=0 -0.03745 -0.16 rpy=0 0 0, axis 0 1 0, limit lower=-10 upper=10 effort=1000 velocity=1000
- added joint rh_ankle: type fixed, parent rh_lower_leg, child rh_foot, origin xyz=0 0 -0.16 rpy=0 0 0, limit lower=-10 upper=10 effort=1000 velocity=1000
- added joint rh_haa_joint: type revolute, parent trunk, child rh_hip_assembly, origin xyz=-0.19 -0.1046 0 rpy=0 0 0, axis 1 0 0, limit lower=-10 upper=10 effort=1000 velocity=1000
- added joint rh_hfe_joint: type revolute, parent rh_hip_assembly, child rh_upper_leg, origin xyz=0 0 0 rpy=0 0 0, axis 0 1 0, limit lower=-10 upper=10 effort=1000 velocity=1000
- added joint rh_kfe_joint: type revolute, parent rh_upper_leg, child rh_lower_leg, origin xyz=0 -0.03745 -0.16 rpy=0 0 0, axis 0 1 0, limit lower=-10 upper=10 effort=1000 velocity=1000
