Commit message: added support for UR5 robot! updated readme after uploading robot URDF descriptions to github

File: robot_urdf/solo.urdf (robot description, URDF)
Before this commit: robot solo, 23 links, 22 joints
Links:
- removed link back_wheel
- removed link front_wheel
- removed link left_wheel
- removed link right_wheel
Joints:
- removed joint z_back_wheel_joint
- removed joint z_front_wheel_joint
- removed joint z_left_wheel_joint
- removed joint z_right_wheel_joint
- joint lf_haa_joint: limit lower=-10 upper=10 effort=1000 velocity=1000 -> lower=-1.30899694 upper=2.44346095 effort=1.2 velocity=58.17764173
- joint lf_hfe_joint: limit lower=-10 upper=10 effort=1000 velocity=1000 -> lower=-3.92699082 upper=1.57079633 effort=1.2 velocity=58.17764173
- joint lf_kfe_joint: limit lower=-10 upper=10 effort=1000 velocity=1000 -> lower=-6.45771823 upper=6.45771823 effort=1.2 velocity=58.17764173
- joint lh_haa_joint: limit lower=-10 upper=10 effort=1000 velocity=1000 -> lower=-1.30899694 upper=2.44346095 effort=1.2 velocity=58.17764173
- joint lh_hfe_joint: limit lower=-10 upper=10 effort=1000 velocity=1000 -> lower=-1.57079633 upper=3.92699082 effort=1.2 velocity=58.17764173
- joint lh_kfe_joint: limit lower=-10 upper=10 effort=1000 velocity=1000 -> lower=-6.45771823 upper=6.45771823 effort=1.2 velocity=58.17764173
- joint rf_haa_joint: limit lower=-10 upper=10 effort=1000 velocity=1000 -> lower=-2.44346095 upper=1.30899694 effort=1.2 velocity=58.17764173
- joint rf_hfe_joint: limit lower=-10 upper=10 effort=1000 velocity=1000 -> lower=-3.92699082 upper=1.57079633 effort=1.2 velocity=58.17764173
- joint rf_kfe_joint: limit lower=-10 upper=10 effort=1000 velocity=1000 -> lower=-6.45771823 upper=6.45771823 effort=1.2 velocity=58.17764173
- joint rh_haa_joint: limit lower=-10 upper=10 effort=1000 velocity=1000 -> lower=-2.44346095 upper=1.30899694 effort=1.2 velocity=58.17764173
- joint rh_hfe_joint: limit lower=-10 upper=10 effort=1000 velocity=1000 -> lower=-1.57079633 upper=3.92699082 effort=1.2 velocity=58.17764173
- joint rh_kfe_joint: limit lower=-10 upper=10 effort=1000 velocity=1000 -> lower=-6.45771823 upper=6.45771823 effort=1.2 velocity=58.17764173

File: robot_urdf/ur5.urdf (robot description, URDF)
Before this commit: robot ur5, 11 links, 10 joints
Links:
- removed link ee_link
- added link base_link_inertia, mass 4.0; collision mesh filename=package://ur_description/meshes/ur5e/collision/base.stl; visual mesh filename=package://ur_description/meshes/ur5e/visual/base.dae
- added link flange
- link base_link: mass 4.0 -> None; geometry 
- link forearm_link: geometry collision mesh filename=package://ur_description/meshes/ur5e/collision/forearm.stl; visual mesh filename=package://ur_description/meshes/ur5e/visual/forearm.dae
- link shoulder_link: geometry collision mesh filename=package://ur_description/meshes/ur5e/collision/shoulder.stl; visual mesh filename=package://ur_description/meshes/ur5e/visual/shoulder.dae
- link tool0: geometry 
- link upper_arm_link: geometry collision mesh filename=package://ur_description/meshes/ur5e/collision/upperarm.stl; visual mesh filename=package://ur_description/meshes/ur5e/visual/upperarm.dae
- link wrist_1_link: geometry collision mesh filename=package://ur_description/meshes/ur5e/collision/wrist1.stl; visual mesh filename=package://ur_description/meshes/ur5e/visual/wrist1.dae
- link wrist_2_link: geometry collision mesh filename=package://ur_description/meshes/ur5e/collision/wrist2.stl; visual mesh filename=package://ur_description/meshes/ur5e/visual/wrist2.dae
- link wrist_3_link: geometry collision mesh filename=package://ur_description/meshes/ur5e/collision/wrist3.stl; visual mesh filename=package://ur_description/meshes/ur5e/visual/wrist3.dae
Joints:
- removed joint ee_fixed_joint
- removed joint wrist_3_link-tool0_fixed_joint
- added joint base_link-base_link_inertia: type fixed, parent base_link, child base_link_inertia, origin xyz=0 0 0 rpy=3.14159265359 0 0
- added joint flange-tool0: type fixed, parent flange, child tool0, origin xyz=0 0 0 rpy=1.57079632679 0 1.57079632679
- added joint wrist_3-flange: type fixed, parent wrist_3_link, child flange, origin xyz=0 0 0 rpy=0 -1.57079632679 -1.57079632679
- joint base_link-base_fixed_joint: origin xyz=0 0 0 rpy=0 0 -3.14159265 -> xyz=0 0 0 rpy=0 0 3.14159265359
- joint elbow_joint: axis 0 1 0 -> 0 0 1; limit lower=-3.14159265 upper=3.14159265 effort=150.0 velocity=3.15 -> lower=-3.14 upper=3.14 effort=150.0 velocity=3.14; origin xyz=0.0 -0.1197 0.425 rpy=0.0 0.0 0.0 -> xyz=-0.425 0 0 rpy=0 0 0
- joint shoulder_lift_joint: axis 0 1 0 -> 0 0 1; limit lower=-3.14159265 upper=3.14159265 effort=150.0 velocity=3.15 -> lower=-6.28 upper=6.28 effort=150.0 velocity=3.14; origin xyz=0.0 0.13585 0.0 rpy=0.0 1.570796325 0.0 -> xyz=0 0 0 rpy=1.570796327 0 0
- joint shoulder_pan_joint: limit lower=-3.14159265 upper=3.14159265 effort=150.0 velocity=3.15 -> lower=-6.28 upper=6.28 effort=150.0 velocity=3.14; origin xyz=0.0 0.0 0.089159 rpy=0.0 0.0 0.0 -> xyz=0 0 0.1625 rpy=0 0 0; parent base_link -> base_link_inertia
- joint world_joint: origin xyz=0.0 0.0 0.0 rpy=0.0 0.0 0.0 -> xyz=0 0 0 rpy=0 0 0
- joint wrist_1_joint: axis 0 1 0 -> 0 0 1; limit lower=-3.14159265 upper=3.14159265 effort=28.0 velocity=3.2 -> lower=-6.28 upper=6.28 effort=28.0 velocity=3.14; origin xyz=0.0 0.0 0.39225 rpy=0.0 1.570796325 0.0 -> xyz=-0.3922 0 0.1333 rpy=0 0 0
- joint wrist_2_joint: limit lower=-3.14159265 upper=3.14159265 effort=28.0 velocity=3.2 -> lower=-6.28 upper=6.28 effort=28.0 velocity=3.14; origin xyz=0.0 0.093 0.0 rpy=0.0 0.0 0.0 -> xyz=0 -0.0997 -2.0448811823e-11 rpy=1.570796327 0 0
- joint wrist_3_joint: axis 0 1 0 -> 0 0 1; limit lower=-3.14159265 upper=3.14159265 effort=28.0 velocity=3.2 -> lower=-6.28 upper=6.28 effort=28.0 velocity=3.14; origin xyz=0.0 0.0 0.09465 rpy=0.0 0.0 0.0 -> xyz=0 0.0996 -2.04283014801e-11 rpy=1.57079632659 3.14159265359 3.14159265359
