Commit message: all labs work again (except L7), allowing the use of separate urdfs for labs (frame ee_link) and ur_description (frame tool0), the generated urdf is placed in robot_urdfs/generate_urdf instead of robot_urdfs

File: robot_urdf/ur5.urdf (robot description, URDF)
Before this commit: robot ur_robot_gazebo, 12 links, 11 joints
Links:
- removed link base_link_inertia
- removed link flange
- added link ee_link; collision box size=0.01 0.01 0.01
- link base_link: mass None -> 4.0; geometry collision mesh filename=package://example-robot-data/robots/ur_description/meshes/u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; visual mesh filename=package://example-robot-data/robots/ur_description/meshes/u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
- link forearm_link: geometry collision mesh filename=package://example-robot-data/robots/ur_description/meshes/u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; visual mesh filename=package://example-robot-data/robots/ur_description/meshes/u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
- link shoulder_link: geometry collision mesh filename=package://example-robot-data/robots/ur_description/meshes/u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; visual mesh filename=package://example-robot-data/robots/ur_description/meshes/u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
- link tool0: geometry collision box size=0.005 0.02 0.05; collision box size=0.005 0.02 0.05
- link upper_arm_link: geometry collision mesh filename=package://example-robot-data/robots/ur_description/meshes/u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; visual mesh filename=package://example-robot-data/robots/ur_description/meshes/u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
- link wrist_1_link: geometry collision mesh filename=package://example-robot-data/robots/ur_description/meshes/u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; visual mesh filename=package://example-robot-data/robots/ur_description/meshes/u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
- link wrist_2_link: geometry collision mesh filename=package://example-robot-data/robots/ur_description/meshes/u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; visual mesh filename=package://example-robot-data/robots/ur_description/meshes/u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
- link wrist_3_link: geometry collision mesh filename=package://example-robot-data/robots/ur_description/meshes/u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; visual mesh filename=package://example-robot-data/robots/ur_description/meshes/u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
Joints:
- removed joint base_link-base_link_inertia
- removed joint flange-tool0
- removed joint wrist_3-flange
- added joint ee_fixed_joint: type fixed, parent wrist_3_link, child ee_link, origin xyz=0.0 0.0823 0.0 rpy=0.0 0.0 1.570796325
- added joint wrist_3_link-tool0_fixed_joint: type fixed, parent wrist_3_link, child tool0, origin xyz=0 0.0823 0 rpy=-1.570796325 0 0
- joint base_link-base_fixed_joint: origin xyz=0 0 0 rpy=0 0 3.14159265359 -> xyz=0 0 0 rpy=0 0 -3.14159265
- joint elbow_joint: axis 0 0 1 -> 0 1 0; limit lower=-3.14 upper=3.14 effort=150.0 velocity=3.14 -> lower=-3.14159265 upper=3.14159265 effort=150.0 velocity=3.15; origin xyz=-0.425 0 0 rpy=0 0 0 -> xyz=0.0 -0.1197 0.425 rpy=0.0 0.0 0.0
- joint shoulder_lift_joint: axis 0 0 1 -> 0 1 0; limit lower=-6.28 upper=6.28 effort=150.0 velocity=3.14 -> lower=-3.14159265 upper=3.14159265 effort=150.0 velocity=3.15; origin xyz=0 0 0 rpy=1.570796327 0 0 -> xyz=0.0 0.13585 0.0 rpy=0.0 1.570796325 0.0
- joint shoulder_pan_joint: limit lower=-6.28 upper=6.28 effort=150.0 velocity=3.14 -> lower=-3.14159265 upper=3.14159265 effort=150.0 velocity=3.15; origin xyz=0 0 0.1625 rpy=0 0 0 -> xyz=0.0 0.0 0.089159 rpy=0.0 0.0 0.0; parent base_link_inertia -> base_link
- joint world_joint: origin xyz=0 0 0 rpy=0 0 0 -> xyz=0.0 0.0 0.0 rpy=0.0 0.0 0.0
- joint wrist_1_joint: axis 0 0 1 -> 0 1 0; limit lower=-6.28 upper=6.28 effort=28.0 velocity=3.14 -> lower=-3.14159265 upper=3.14159265 effort=28.0 velocity=3.2; origin xyz=-0.3922 0 0.1333 rpy=0 0 0 -> xyz=0.0 0.0 0.39225 rpy=0.0 1.570796325 0.0
- joint wrist_2_joint: limit lower=-6.28 upper=6.28 effort=28.0 velocity=3.14 -> lower=-3.14159265 upper=3.14159265 effort=28.0 velocity=3.2; origin xyz=0 -0.0997 -2.0448811823e-11 rpy=1.570796327 0 0 -> xyz=0.0 0.093 0.0 rpy=0.0 0.0 0.0
- joint wrist_3_joint: axis 0 0 1 -> 0 1 0; limit lower=-6.28 upper=6.28 effort=28.0 velocity=3.14 -> lower=-3.14159265 upper=3.14159265 effort=28.0 velocity=3.2; origin xyz=0 0.0996 -2.04283014801e-11 rpy=1.57079632659 3.14159265359 3.14159265359 -> xyz=0.0 0.0 0.09465 rpy=0.0 0.0 0.0
