Commit message: now using only visualize.launch not anymore visualize_robotName.launch
updated urdfs in robot_urdf folder
packed labs in a folder

File: robot_urdf/aliengo.urdf (robot description, URDF)
Before this commit: robot aliengo, 19 links, 18 joints
Links:
- removed link lf_hipassembly
- removed link lh_hipassembly
- removed link rf_hipassembly
- removed link rh_hipassembly
- added link lf_hip, mass 1.993; collision cylinder length=0.0418 radius=0.046; visual mesh filename=package://aliengo_description/meshes/hip.dae scale=1 1 1
- added link lh_hip, mass 1.993; collision cylinder length=0.0418 radius=0.046; visual mesh filename=package://aliengo_description/meshes/hip.dae scale=1 1 1
- added link rf_hip, mass 1.993; collision cylinder length=0.0418 radius=0.046; visual mesh filename=package://aliengo_description/meshes/hip.dae scale=1 1 1
- added link rh_hip, mass 1.993; collision cylinder length=0.0418 radius=0.046; visual mesh filename=package://aliengo_description/meshes/hip.dae scale=1 1 1
- added link trunk_imu, mass 0.001; collision box size=.001 .001 .001; visual box size=0.001 0.001 0.001
- link base_link: geometry 
- link lf_foot: mass None -> 0.06; geometry collision sphere radius=0.0265; visual sphere radius=0.0165
- link lf_lowerleg: mass 0.267 -> 0.207; geometry collision box size=0.25 0.0208 0.016; visual mesh filename=package://aliengo_description/meshes/calf.dae scale=1 1 1
- link lf_upperleg: geometry collision box size=0.25 0.0374 0.043; visual mesh filename=package://aliengo_description/meshes/thigh.dae scale=1 1 1
- link lh_foot: mass None -> 0.06; geometry collision sphere radius=0.0265; visual sphere radius=0.0165
- link lh_lowerleg: mass 0.267 -> 0.207; geometry collision box size=0.25 0.0208 0.016; visual mesh filename=package://aliengo_description/meshes/calf.dae scale=1 1 1
- link lh_upperleg: geometry collision box size=0.25 0.0374 0.043; visual mesh filename=package://aliengo_description/meshes/thigh.dae scale=1 1 1
- link rf_foot: mass None -> 0.06; geometry collision sphere radius=0.0265; visual sphere radius=0.0165
- link rf_lowerleg: mass 0.267 -> 0.207; geometry collision box size=0.25 0.0208 0.016; visual mesh filename=package://aliengo_description/meshes/calf.dae scale=1 1 1
- link rf_upperleg: geometry collision box size=0.25 0.0374 0.043; visual mesh filename=package://aliengo_description/meshes/thigh_mirror.dae scale=1 1 1
- link rh_foot: mass None -> 0.06; geometry collision sphere radius=0.0265; visual sphere radius=0.0165
- link rh_lowerleg: mass 0.267 -> 0.207; geometry collision box size=0.25 0.0208 0.016; visual mesh filename=package://aliengo_description/meshes/calf.dae scale=1 1 1
- link rh_upperleg: geometry collision box size=0.25 0.0374 0.043; visual mesh filename=package://aliengo_description/meshes/thigh_mirror.dae scale=1 1 1
- link trunk: mass 18.041 -> 11.041; geometry collision box size=0.647 0.15 0.112; visual mesh filename=package://aliengo_description/meshes/trunk.dae scale=1 1 1
Joints:
- removed joint lf_foot_joint
- removed joint lh_foot_joint
- removed joint rf_foot_joint
- removed joint rh_foot_joint
- added joint imu_joint: type fixed, parent trunk, child trunk_imu, origin xyz=0 0 0 rpy=0 0 0
- added joint lf_foot_fixed: type fixed, parent lf_lowerleg, child lf_foot, origin xyz=0 0 -0.25 rpy=0 0 0
- added joint lh_foot_fixed: type fixed, parent lh_lowerleg, child lh_foot, origin xyz=0 0 -0.25 rpy=0 0 0
- added joint rf_foot_fixed: type fixed, parent rf_lowerleg, child rf_foot, origin xyz=0 0 -0.25 rpy=0 0 0
- added joint rh_foot_fixed: type fixed, parent rh_lowerleg, child rh_foot, origin xyz=0 0 -0.25 rpy=0 0 0
- joint lf_haa_joint: axis 0 0 1 -> 1 0 0; child lf_hipassembly -> lf_hip; limit lower=-1.2217304764 upper=1.2217304764 effort=44.0 velocity=20.0 -> lower=-1.2217304763960306 upper=1.2217304763960306 effort=44 velocity=20; origin xyz=0.2399 0.051 0 rpy=3.14159265359 1.57079632679 0 -> xyz=0.2399 0.051 0 rpy=0 0 0
- joint lf_hfe_joint: axis 0 0 1 -> 0 1 0; limit lower=-6.28318530718 upper=6.28318530718 effort=44.0 velocity=20.0 -> lower=-3.141592653589793 upper=3.141592653589793 effort=44 velocity=20; origin xyz=0 -0.083 0 rpy=1.57079632679 0 0 -> xyz=0 0.083 0 rpy=0 0 0; parent lf_hipassembly -> lf_hip
- joint lf_kfe_joint: axis 0 0 1 -> 0 1 0; limit lower=-2.77507351067 upper=-0.645771823238 effort=55.0 velocity=16.0 -> lower=-2.775073510670984 upper=-0.6457718232379019 effort=55 velocity=16; origin xyz=0.25 0 0 rpy=0 0 0 -> xyz=0 0 -0.25 rpy=0 0 0
- joint lh_haa_joint: axis 0 0 1 -> 1 0 0; child lh_hipassembly -> lh_hip; limit lower=-1.2217304764 upper=1.2217304764 effort=44.0 velocity=20.0 -> lower=-1.2217304763960306 upper=1.2217304763960306 effort=44 velocity=20; origin xyz=-0.2399 0.051 0 rpy=3.14159265359 1.57079632679 0 -> xyz=-0.2399 0.051 0 rpy=0 0 0
- joint lh_hfe_joint: axis 0 0 1 -> 0 1 0; limit lower=-6.28318530718 upper=6.28318530718 effort=44.0 velocity=20.0 -> lower=-3.141592653589793 upper=3.141592653589793 effort=44 velocity=20; origin xyz=0 -0.083 0 rpy=1.57079632679 0 0 -> xyz=0 0.083 0 rpy=0 0 0; parent lh_hipassembly -> lh_hip
- joint lh_kfe_joint: axis 0 0 1 -> 0 1 0; limit lower=-2.77507351067 upper=-0.645771823238 effort=55.0 velocity=16.0 -> lower=-2.775073510670984 upper=-0.6457718232379019 effort=55 velocity=16; origin xyz=0.25 0 0 rpy=0 0 0 -> xyz=0 0 -0.25 rpy=0 0 0
- joint rf_haa_joint: axis 0 0 1 -> 1 0 0; child rf_hipassembly -> rf_hip; limit lower=-1.2217304764 upper=1.2217304764 effort=44.0 velocity=20.0 -> lower=-1.2217304763960306 upper=1.2217304763960306 effort=44 velocity=20; origin xyz=0.2399 -0.051 0 rpy=0 1.57079632679 0 -> xyz=0.2399 -0.051 0 rpy=0 0 0
- joint rf_hfe_joint: axis 0 0 1 -> 0 1 0; limit lower=-6.28318530718 upper=6.28318530718 effort=44.0 velocity=20.0 -> lower=-3.141592653589793 upper=3.141592653589793 effort=44 velocity=20; origin xyz=0 -0.083 0 rpy=-1.57079632679 0 0 -> xyz=0 -0.083 0 rpy=0 0 0; parent rf_hipassembly -> rf_hip
- joint rf_kfe_joint: axis 0 0 1 -> 0 1 0; limit lower=-2.77507351067 upper=-0.645771823238 effort=55.0 velocity=16.0 -> lower=-2.775073510670984 upper=-0.6457718232379019 effort=55 velocity=16; origin xyz=0.25 0 0 rpy=0 0 0 -> xyz=0 0 -0.25 rpy=0 0 0
- joint rh_haa_joint: axis 0 0 1 -> 1 0 0; child rh_hipassembly -> rh_hip; limit lower=-1.2217304764 upper=1.2217304764 effort=44.0 velocity=20.0 -> lower=-1.2217304763960306 upper=1.2217304763960306 effort=44 velocity=20; origin xyz=-0.2399 -0.051 0 rpy=0 1.57079632679 0 -> xyz=-0.2399 -0.051 0 rpy=0 0 0
- joint rh_hfe_joint: axis 0 0 1 -> 0 1 0; limit lower=-6.28318530718 upper=6.28318530718 effort=44.0 velocity=20.0 -> lower=-3.141592653589793 upper=3.141592653589793 effort=44 velocity=20; origin xyz=0 -0.083 0 rpy=-1.57079632679 0 0 -> xyz=0 -0.083 0 rpy=0 0 0; parent rh_hipassembly -> rh_hip
- joint rh_kfe_joint: axis 0 0 1 -> 0 1 0; limit lower=-2.77507351067 upper=-0.645771823238 effort=55.0 velocity=16.0 -> lower=-2.775073510670984 upper=-0.6457718232379019 effort=55 velocity=16; origin xyz=0.25 0 0 rpy=0 0 0 -> xyz=0 0 -0.25 rpy=0 0 0

File: robot_urdf/double_pendulum.urdf (robot description, URDF)
Before this commit: robot 2dof_planar, 3 links, 2 joints
Links:
- link base_link: geometry collision mesh filename=package://example-robot-data/robots/double_pendulum_descrip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; visual mesh filename=package://example-robot-data/robots/double_pendulum_descrip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
- link link1: geometry collision mesh filename=package://example-robot-data/robots/double_pendulum_descrip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; visual mesh filename=package://example-robot-data/robots/double_pendulum_descrip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
- link link2: geometry collision mesh filename=package://example-robot-data/robots/double_pendulum_descrip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; visual mesh filename=package://example-robot-data/robots/double_pendulum_descrip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

File: robot_urdf/hyq.urdf (robot description, URDF)
Before this commit: robot hyq, 19 links, 18 joints
Joints:
- joint lf_foot_joint: origin xyz=0.341 0 0 rpy=1.57079632679 0 -1.57079632679 -> xyz=0.341 0 0 rpy=1.5707963267948966 0 -1.5707963267948966
- joint lf_haa_joint: limit lower=-1.2217304764 upper=0.436332312999 effort=150 velocity=12.0 -> lower=-1.2217304763960306 upper=0.4363323129985824 effort=150 velocity=12.0; origin xyz=0.3735 0.207 0 rpy=0 1.57079632679 3.14159265359 -> xyz=0.3735 0.207 0 rpy=0 1.5707963267948966 3.141592653589793
- joint lf_hfe_joint: limit lower=-0.872664625997 upper=1.2217304764 effort=150 velocity=12.0 -> lower=-0.8726646259971648 upper=1.2217304763960306 effort=150 velocity=12.0; origin xyz=0.08 0 0 rpy=1.57079632679 0 0 -> xyz=0.08 0 0 rpy=1.5707963267948966 0 0
- joint lf_kfe_joint: limit lower=-2.44346095279 upper=-0.349065850399 effort=150 velocity=12.0 -> lower=-2.443460952792061 upper=-0.3490658503988659 effort=150 velocity=12.0
- joint lh_foot_joint: origin xyz=0.341 0 0 rpy=1.57079632679 0 -1.57079632679 -> xyz=0.341 0 0 rpy=1.5707963267948966 0 -1.5707963267948966
- joint lh_haa_joint: limit lower=-1.2217304764 upper=0.436332312999 effort=150 velocity=12.0 -> lower=-1.2217304763960306 upper=0.4363323129985824 effort=150 velocity=12.0; origin xyz=-0.3735 0.207 0 rpy=0 1.57079632679 3.14159265359 -> xyz=-0.3735 0.207 0 rpy=0 1.5707963267948966 3.141592653589793
- joint lh_hfe_joint: limit lower=-1.2217304764 upper=0.872664625997 effort=150 velocity=12.0 -> lower=-1.2217304763960306 upper=0.8726646259971648 effort=150 velocity=12.0; origin xyz=0.08 0 0 rpy=1.57079632679 0 0 -> xyz=0.08 0 0 rpy=1.5707963267948966 0 0
- joint lh_kfe_joint: limit lower=0.349065850399 upper=2.44346095279 effort=150 velocity=12.0 -> lower=0.3490658503988659 upper=2.443460952792061 effort=150 velocity=12.0
- joint rf_foot_joint: origin xyz=0.341 0 0 rpy=1.57079632679 0 -1.57079632679 -> xyz=0.341 0 0 rpy=1.5707963267948966 0 -1.5707963267948966
- joint rf_haa_joint: limit lower=-1.2217304764 upper=0.436332312999 effort=150 velocity=12.0 -> lower=-1.2217304763960306 upper=0.4363323129985824 effort=150 velocity=12.0; origin xyz=0.3735 -0.207 0 rpy=0 1.57079632679 0 -> xyz=0.3735 -0.207 0 rpy=0 1.5707963267948966 0
- joint rf_hfe_joint: limit lower=-0.872664625997 upper=1.2217304764 effort=150 velocity=12.0 -> lower=-0.8726646259971648 upper=1.2217304763960306 effort=150 velocity=12.0; origin xyz=0.08 0 0 rpy=-1.57079632679 0 0 -> xyz=0.08 0 0 rpy=-1.5707963267948966 0 0
- joint rf_kfe_joint: limit lower=-2.44346095279 upper=-0.349065850399 effort=150 velocity=12.0 -> lower=-2.443460952792061 upper=-0.3490658503988659 effort=150 velocity=12.0
- joint rh_foot_joint: origin xyz=0.341 0 0 rpy=1.57079632679 0 -1.57079632679 -> xyz=0.341 0 0 rpy=1.5707963267948966 0 -1.5707963267948966
- joint rh_haa_joint: limit lower=-1.2217304764 upper=0.436332312999 effort=150 velocity=12.0 -> lower=-1.2217304763960306 upper=0.4363323129985824 effort=150 velocity=12.0; origin xyz=-0.3735 -0.207 0 rpy=0 1.57079632679 0 -> xyz=-0.3735 -0.207 0 rpy=0 1.5707963267948966 0
- joint rh_hfe_joint: limit lower=-1.2217304764 upper=0.872664625997 effort=150 velocity=12.0 -> lower=-1.2217304763960306 upper=0.8726646259971648 effort=150 velocity=12.0; origin xyz=0.08 0 0 rpy=-1.57079632679 0 0 -> xyz=0.08 0 0 rpy=-1.5707963267948966 0 0
- joint rh_kfe_joint: limit lower=0.349065850399 upper=2.44346095279 effort=150 velocity=12.0 -> lower=0.3490658503988659 upper=2.443460952792061 effort=150 velocity=12.0

File: robot_urdf/jumpleg.urdf (robot description, URDF)
Before this commit: robot jumpleg, 9 links, 8 joints
Joints:
- joint base_x_joint: limit lower=-100 upper=100 effort=150 velocity=100.0 -> lower=-100 upper=100 effort=1000 velocity=100.0
- joint base_y_joint: limit lower=-100 upper=100 effort=150 velocity=100.0 -> lower=-100 upper=100 effort=1000 velocity=100.0
- joint base_z_joint: limit lower=-100 upper=100 effort=150 velocity=100.0 -> lower=-100 upper=100 effort=1000 velocity=100.0
- joint lf_haa_joint: limit lower=-1.30899694 upper=2.44346095 effort=1.2 velocity=58.17764173 -> lower=-1.30899694 upper=2.44346095 effort=10 velocity=58.17764173
- joint lf_hfe_joint: limit lower=-3.92699082 upper=1.57079633 effort=1.2 velocity=58.17764173 -> lower=-3.92699082 upper=1.57079633 effort=10 velocity=58.17764173
- joint lf_kfe_joint: limit lower=-6.45771823 upper=6.45771823 effort=1.2 velocity=58.17764173 -> lower=-6.45771823 upper=6.45771823 effort=10 velocity=58.17764173

File: robot_urdf/solo_fw.urdf (robot description, URDF)
Before this commit: robot solo, 19 links, 18 joints
Links:
- added link left_wheel, mass 0.1; collision mesh filename=package://solo_description/meshes/stl/flywheel/flywheel.stl scale=0.001 0.001 0.001; visual mesh filename=package://solo_description/meshes/stl/flywheel/flywheel.stl scale=0.001 0.001 0.001
- added link right_wheel, mass 0.1; collision mesh filename=package://solo_description/meshes/stl/flywheel/flywheel.stl scale=0.001 0.001 0.001; visual mesh filename=package://solo_description/meshes/stl/flywheel/flywheel.stl scale=0.001 0.001 0.001
Joints:
- added joint z_left_wheel_joint: type revolute, parent trunk, child left_wheel, origin xyz=0.0 0.067 0.066 rpy=-1.5707963267948966 0 -0.0, axis 0 0 1, limit lower=-1e06 upper=1e06 effort=0.225 velocity=523
- added joint z_right_wheel_joint: type revolute, parent trunk, child right_wheel, origin xyz=0.0 -0.067 0.066 rpy=1.5707963267948966 0 0.0, axis 0 0 1, limit lower=-1e06 upper=1e06 effort=0.225 velocity=523
